Commit message: aruco_detect ok!!

File: src/car_description/carA/box.xacro (robot description, xacro)
@@ -21,5 +21,5 @@
   </link>
   <gazebo reference="box_link">
-    <material>SOLab/aruco200</material>
+    <material>Yulin/fucface</material>
   </gazebo>
 </robot>

File: src/car_description/carA/carA.xacro (robot description, xacro)
@@ -7,5 +7,5 @@
     <parent link="carA__base_link"/>
     <child link="carA__link_1"/>
-    <origin rpy="0       0       0" xyz="0.425 0.225  0.076"/>
+    <origin rpy="0       0       0" xyz="0.425 0.225  0.08"/>
     <axis xyz="0  0  0"/>
   </joint>
@@ -13,5 +13,5 @@
     <parent link="carA__base_link"/>
     <child link="carA__link_1_clone"/>
-    <origin rpy="0       0       0" xyz="0.425   -0.225  0.076"/>
+    <origin rpy="0       0       0" xyz="0.425   -0.225  0.08"/>
     <axis xyz="0  0  0"/>
   </joint>
@@ -19,5 +19,5 @@
     <parent link="carA__base_link"/>
     <child link="carA__link_1_clone_0"/>
-    <origin rpy="0       0       0" xyz="-0.425  -0.225  0.076"/>
+    <origin rpy="0       0       0" xyz="-0.425  -0.225  0.08"/>
     <axis xyz="0  0  0"/>
   </joint>
@@ -25,5 +25,5 @@
     <parent link="carA__base_link"/>
     <child link="carA__link_1_clone_1"/>
-    <origin rpy="0       0       0" xyz="-0.425  0.225  0.076"/>
+    <origin rpy="0       0       0" xyz="-0.425  0.225  0.08"/>
     <axis xyz="0  0  0"/>
   </joint>
@@ -82,11 +82,11 @@
       <origin rpy="0  0  0" xyz="0  0  0"/>
       <geometry>
-        <sphere radius="0.075"/>
-      </geometry>
-    </collision>
-    <visual>
-      <origin rpy="0  0  0" xyz="0  0  0"/>
-      <geometry>
-        <sphere radius="0.075"/>
+        <sphere radius="0.07"/>
+      </geometry>
+    </collision>
+    <visual>
+      <origin rpy="0  0  0" xyz="0  0  0"/>
+      <geometry>
+        <sphere radius="0.07"/>
       </geometry>
     </visual>
@@ -101,11 +101,11 @@
       <origin rpy="0  0  0" xyz="0  0  0"/>
       <geometry>
-        <sphere radius="0.075"/>
-      </geometry>
-    </collision>
-    <visual>
-      <origin rpy="0  0  0" xyz="0  0  0"/>
-      <geometry>
-        <sphere radius="0.075"/>
+        <sphere radius="0.07"/>
+      </geometry>
+    </collision>
+    <visual>
+      <origin rpy="0  0  0" xyz="0  0  0"/>
+      <geometry>
+        <sphere radius="0.07"/>
       </geometry>
     </visual>
@@ -120,11 +120,11 @@
       <origin rpy="0  0  0" xyz="0  0  0"/>
       <geometry>
-        <sphere radius="0.075"/>
-      </geometry>
-    </collision>
-    <visual>
-      <origin rpy="0  0  0" xyz="0  0  0"/>
-      <geometry>
-        <sphere radius="0.075"/>
+        <sphere radius="0.07"/>
+      </geometry>
+    </collision>
+    <visual>
+      <origin rpy="0  0  0" xyz="0  0  0"/>
+      <geometry>
+        <sphere radius="0.07"/>
       </geometry>
     </visual>
@@ -139,11 +139,11 @@
       <origin rpy="0  0  0" xyz="0  0  0"/>
       <geometry>
-        <sphere radius="0.075"/>
-      </geometry>
-    </collision>
-    <visual>
-      <origin rpy="0  0  0" xyz="0  0  0"/>
-      <geometry>
-        <sphere radius="0.075"/>
+        <sphere radius="0.07"/>
+      </geometry>
+    </collision>
+    <visual>
+      <origin rpy="0  0  0" xyz="0  0  0"/>
+      <geometry>
+        <sphere radius="0.07"/>
       </geometry>
     </visual>

Commit message: debug texture

File: src/car_description/carA/box.xacro (robot description, xacro)
@@ -21,5 +21,5 @@
   </link>
   <gazebo reference="box_link">
-    <material>Yulin/fucface</material>
+    <material>test/aruco</material>
   </gazebo>
 </robot>

Commit message: fiducial - tf code ok!!

File: src/car_description/carA/box.xacro (robot description, xacro)
@@ -21,5 +21,5 @@
   </link>
   <gazebo reference="box_link">
-    <material>test/aruco</material>
+    <material>test/aruco50</material>
   </gazebo>
 </robot>
