Commit message: add aruco box in gazebo

File: src/car_description/carA/carA.xacro (robot description, xacro)
@@ -56,7 +56,7 @@
   <link name="carA__base_link">
     <inertial>
-      <mass value="10"/>
-      <origin rpy="0  0  0" xyz="0  0  0"/>
-      <inertia ixx="1.66667" ixy="0" ixz="0" iyy="1.66667" iyz="0" izz="1.66667"/>
+      <mass value="50"/>
+      <origin rpy="0  0  0" xyz="0  0  0"/>
+      <inertia ixx="1.875" ixy="0" ixz="0" iyy="4.541667" iyz="0" izz="5.6667"/>
     </inertial>
     <collision name="carA__collision">

Commit message: finish model

File: src/car_description/carA/carA.xacro (robot description, xacro)
@@ -197,5 +197,5 @@
       <origin rpy="0  0  0" xyz="0  0  0"/>
       <geometry>
-        <mesh filename="home/yulin/carA_sim_ws/src/car_description/carA/meshes/hokuyo.dae" scale="0.050 0.050 0.050"/>
+        <mesh filename="package://car_description/carA/meshes/hokuyo.dae" />
       </geometry>
     </visual>
@@ -210,5 +210,5 @@
       <origin rpy="0  0  0" xyz="0  0  0"/>
       <geometry>
-        <mesh filename="package://car_description/meshes/hokuyo.dae" scale="0.050 0.050 0.050"/>
+        <mesh filename="package://car_description/carA/meshes/hokuyo.dae" />
       </geometry>
     </visual>
@@ -217,7 +217,7 @@
   <link name="camera">
       <visual>
-        <origin xyz="0 0 0" rpy="0 0 0"/>
+        <origin xyz="-0.015 0 -0.0257" rpy="1.5707 0 0"/>
         <geometry>
-            <mesh filename="package://car_description/meshes/hokuyo.dae" scale="0.050 0.050 0.050"/>
+            <mesh filename="package://car_description/carA/meshes/webcam.stl" scale="0.01 0.01 0.01" />
         </geometry>
       </visual>
@@ -240,5 +240,5 @@
         <origin xyz="0 0 0" rpy="0 0 0"/>
         <geometry>
-            <mesh filename="package://car_description/meshes/hokuyo.dae" scale="0.050 0.050 0.050"/>
+            <mesh filename="package://car_description/carA/meshes/hokuyo.dae" scale="0.050 0.050 0.050"/>
         </geometry>
       </visual>
